Commit message: manipulation challenge examples

File: platforms/ur5_ros2_gazebo/urdf/sensors/d435.gazebo.xacro (robot description, xacro)
@@ -31,4 +31,11 @@
             <format>RGB_INT8</format>
           </image>
+          <lens>
+            <intrinsics>
+              <fx>463.8</fx> <fy>463.8</fy>
+              <cx>320.0</cx> <cy>240.0</cy>
+              <s>0</s>
+            </intrinsics>
+          </lens>
           <clip>
             <near>0.1</near>
@@ -91,9 +98,17 @@
       <sensor name="${camera_name}depth" type="depth">
         <camera name="${camera_name}">
-          <horizontal_fov>${85.2*deg_to_rad}</horizontal_fov>
+          <horizontal_fov>${69.4*deg_to_rad}</horizontal_fov>
+          <!-- <horizontal_fov>${85.2*deg_to_rad}</horizontal_fov> -->
           <image>
             <width>640</width>
             <height>480</height>
           </image>
+          <lens>
+            <intrinsics>
+              <fx>463.8</fx> <fy>463.8</fy>
+              <cx>320.0</cx> <cy>240.0</cy>
+              <s>0</s>
+            </intrinsics>
+          </lens>
           <clip>
             <near>0.1</near>

File: platforms/ur5_ros2_gazebo/urdf/sensors/d435.urdf.xacro (robot description, xacro)
@@ -12,5 +12,5 @@
   <xacro:include filename="$(find ur5_ros2_gazebo)/urdf/sensors/d435.gazebo.xacro"/>
   <xacro:macro name="sensor_d435" params="parent *origin name:=camera
-                                          use_nominal_extrinsics:=false
+                                          use_nominal_extrinsics:=true
                                           add_plug:=false
                                           use_mesh:=true
@@ -144,5 +144,7 @@
     </xacro:if>
     <!-- Realsense Gazebo Plugin -->
-    <xacro:gazebo_d435 camera_name="${name}" reference_link="${name}_link" topics_ns="${topics_ns}" depth_optical_frame="${name}_depth_optical_frame" color_optical_frame="${name}_color_optical_frame" infrared1_optical_frame="${name}_left_ir_optical_frame" infrared2_optical_frame="${name}_right_ir_optical_frame" publish_pointcloud="${publish_pointcloud}"/>
+    <!-- Force to use the same depth and optical frame-->
+    <xacro:gazebo_d435 camera_name="${name}" reference_link="${name}_link" topics_ns="${topics_ns}" depth_optical_frame="${name}_color_optical_frame" color_optical_frame="${name}_color_optical_frame" infrared1_optical_frame="${name}_left_ir_optical_frame" infrared2_optical_frame="${name}_right_ir_optical_frame" publish_pointcloud="${publish_pointcloud}"/>
+    <!-- <xacro:gazebo_d435 camera_name="${name}" reference_link="${name}_link" topics_ns="${topics_ns}" depth_optical_frame="${name}_depth_optical_frame" color_optical_frame="${name}_color_optical_frame" infrared1_optical_frame="${name}_left_ir_optical_frame" infrared2_optical_frame="${name}_right_ir_optical_frame" publish_pointcloud="${publish_pointcloud}"/> -->
   </xacro:macro>
 </robot>

File: platforms/ur5_ros2_gazebo/urdf/ur5.urdf.xacro (robot description, xacro)
@@ -131,5 +131,5 @@
       <visual>
         <geometry>
-          <mesh filename="file://$(find robotiq_85_description)/meshes/visual/d435_UR5_camera_mount.dae" scale="0.001 0.001 0.001"/>
+          <mesh filename="file://$(find ur5_ros2_gazebo)/urdf/sensors/meshes/d435_UR5_camera_mount.dae" scale="0.001 0.001 0.001"/>
         </geometry>
       </visual>
@@ -148,5 +148,5 @@
     </link>
     <xacro:sensor_d435 name="wrist_camera" topics_ns="wrist_camera" parent="wrist_camera_base_link" >
-      <origin xyz="0.0 0.08 0.015" rpy="1.575796 -1.575796 0"/>
+      <origin xyz="0.0 0.06 0.015" rpy="-1.575796 -1.575796 0"/>
     </xacro:sensor_d435>
   </xacro:if>
